File: va4.sch (KiCad schematic (older format))
At the start: 12 parts, among them J1 LED, J2 MJ-4PP-9, SW1 RESET_SWITCH, SW2 SW_PUSH, SW3 SW_PUSH, SW4 SW_PUSH, SW5 SW_PUSH, U1 ProMicro

Commit message: Assign footprints to schematic symbols
Parts:
- D1, D2, D3, D4: footprint (none) -> kbd:D3_TH_SMD
- J1: footprint (none) -> kbd:StripLED_rev
- J2: footprint (none) -> kbd:MJ-4PP-9
- SW1: footprint (none) -> kbd:ResetSW
- SW2, SW3, SW4: footprint (none) -> kbd:MX_ALPS_PG1350_noLed
- SW5: footprint (none) -> kbd:MX_ALPS_PG1350_noLed_1.75u
- U1: footprint (none) -> kbd:ProMicro_v2
Changed lines of the file:
@@
 F 0 "U1" H 2725 3937 60  0000 C CNN
 F 1 "ProMicro" H 2725 3831 60  0000 C CNN
-F 2 "" H 2825 1850 60  0000 C CNN
+F 2 "kbd:ProMicro_v2" H 2825 1850 60  0001 C CNN
 F 3 "" H 2825 1850 60  0000 C CNN
 	1    2725 2900
@@
 F 0 "SW1" H 4250 4430 50  0000 C CNN
 F 1 "RESET_SWITCH" H 4250 4339 50  0000 C CNN
-F 2 "" H 4250 4175 50  0000 C CNN
+F 2 "kbd:ResetSW" H 4250 4175 50  0001 C CNN
 F 3 "" H 4250 4175 50  0000 C CNN
 	1    4250 4175
@@
 F 0 "J2" H 2705 4451 50  0000 C CNN
 F 1 "MJ-4PP-9" H 2705 4360 50  0000 C CNN
-F 2 "" H 2950 4350 50  0001 C CNN
+F 2 "kbd:MJ-4PP-9" H 2950 4350 50  0001 C CNN
 F 3 "~" H 2950 4350 50  0001 C CNN
 	1    2675 4175
@@
 F 0 "J1" H 1570 3800 50  0000 C CNN
 F 1 "LED" H 1570 3891 50  0000 C CNN
-F 2 "" H 1650 4125 50  0001 C CNN
+F 2 "kbd:StripLED_rev" H 1650 4125 50  0001 C CNN
 F 3 "~" H 1650 4125 50  0001 C CNN
 	1    1650 4125
@@
 F 0 "SW2" H 5000 2930 50  0000 C CNN
 F 1 "SW_PUSH" H 5000 2839 50  0000 C CNN
-F 2 "" H 5000 2675 50  0000 C CNN
+F 2 "kbd:MX_ALPS_PG1350_noLed" H 5000 2675 50  0001 C CNN
 F 3 "" H 5000 2675 50  0000 C CNN
 	1    5000 2675
@@
 F 0 "D1" V 5346 2746 50  0000 R CNN
 F 1 "D" V 5255 2746 50  0000 R CNN
-F 2 "" H 5300 2825 50  0001 C CNN
+F 2 "kbd:D3_TH_SMD" H 5300 2825 50  0001 C CNN
 F 3 "~" H 5300 2825 50  0001 C CNN
 	1    5300 2825
@@
 F 0 "SW3" H 5900 2930 50  0000 C CNN
 F 1 "SW_PUSH" H 5900 2839 50  0000 C CNN
-F 2 "" H 5900 2675 50  0000 C CNN
+F 2 "kbd:MX_ALPS_PG1350_noLed" H 5900 2675 50  0001 C CNN
 F 3 "" H 5900 2675 50  0000 C CNN
 	1    5900 2675
@@
 F 0 "D2" V 6246 2746 50  0000 R CNN
 F 1 "D" V 6155 2746 50  0000 R CNN
-F 2 "" H 6200 2825 50  0001 C CNN
+F 2 "kbd:D3_TH_SMD" H 6200 2825 50  0001 C CNN
 F 3 "~" H 6200 2825 50  0001 C CNN
 	1    6200 2825
@@
 F 0 "SW4" H 6800 2930 50  0000 C CNN
 F 1 "SW_PUSH" H 6800 2839 50  0000 C CNN
-F 2 "" H 6800 2675 50  0000 C CNN
+F 2 "kbd:MX_ALPS_PG1350_noLed" H 6800 2675 50  0001 C CNN
 F 3 "" H 6800 2675 50  0000 C CNN
 	1    6800 2675
@@
 F 0 "D3" V 7146 2746 50  0000 R CNN
 F 1 "D" V 7055 2746 50  0000 R CNN
-F 2 "" H 7100 2825 50  0001 C CNN
+F 2 "kbd:D3_TH_SMD" H 7100 2825 50  0001 C CNN
 F 3 "~" H 7100 2825 50  0001 C CNN
 	1    7100 2825
@@
 F 0 "SW5" H 7675 2930 50  0000 C CNN
 F 1 "SW_PUSH" H 7675 2839 50  0000 C CNN
-F 2 "" H 7675 2675 50  0000 C CNN
+F 2 "kbd:MX_ALPS_PG1350_noLed_1.75u" H 7675 2675 50  0001 C CNN
 F 3 "" H 7675 2675 50  0000 C CNN
 	1    7675 2675
@@
 F 0 "D4" V 8021 2746 50  0000 R CNN
 F 1 "D" V 7930 2746 50  0000 R CNN
-F 2 "" H 7975 2825 50  0001 C CNN
+F 2 "kbd:D3_TH_SMD" H 7975 2825 50  0001 C CNN
 F 3 "~" H 7975 2825 50  0001 C CNN
 	1    7975 2825

Commit message: Fix 4th key layout for Kailh Choc key switch(low profile)
Parts:
- SW5: footprint kbd:MX_ALPS_PG1350_noLed_1.75u -> kbd:MX_ALPS_PG1350_noLed
Changed lines of the file:
@@
 EESchema Schematic File Version 4
+LIBS:va4-cache
 EELAYER 26 0
 EELAYER END
@@
 F 0 "SW5" H 7675 2930 50  0000 C CNN
 F 1 "SW_PUSH" H 7675 2839 50  0000 C CNN
-F 2 "kbd:MX_ALPS_PG1350_noLed_1.75u" H 7675 2675 50  0001 C CNN
+F 2 "kbd:MX_ALPS_PG1350_noLed" H 7675 2675 50  0001 C CNN
 F 3 "" H 7675 2675 50  0000 C CNN
 	1    7675 2675
